File: DualEncoder/MBRadioPanel.sch (KiCad schematic (older format))
At the start: 16 parts, among them J1 Conn_01x12_Male

Commit message: Add files via upload
Parts:
- removed J1: Conn_01x12_Male, Connector_PinHeader_2.54mm:PinHeader_1x12_P2.54mm_Vertical, symbol Connector:Conn_01x12_Male
- added C5: 4.7µF, Capacitor_SMD:C_0603_1608Metric, symbol Device:C_Small
- added D1: MUTE, LED_SMD:LED_0603_1608Metric_Castellated, symbol Device:LED_Small
- added D2: GP, LED_SMD:LED_0603_1608Metric_Castellated, symbol Device:LED_Small
- added J1: Conn_01x09_Male, Connector_PinHeader_2.54mm:PinHeader_1x09_P2.54mm_Vertical, symbol Connector:Conn_01x09_Male
- added J2: Stemma QT, Connector_JST:JST_SH_BM04B-SRSS-TB_1x04-1MP_P1.00mm_Vertical, symbol Connector:Conn_01x04_Male
- added JB1: Conn_02x03_Odd_Even, Connector_PinHeader_2.00mm:PinHeader_2x03_P2.00mm_Vertical, symbol Connector_Generic:Conn_02x03_Odd_Even
- added JP1: i2C PU, Connector_PinHeader_2.00mm:PinHeader_1x02_P2.00mm_Vertical, symbol Device:Jumper_NO_Small
- added R10, R11, R9: 10kΩ, Resistor_SMD:R_0402_1005Metric, symbol Device:R_Small
- added R12, R13: 1kΩ, Resistor_SMD:R_0402_1005Metric, symbol Device:R_Small
- added R14, R15: 4.7kΩ, Resistor_SMD:R_0402_1005Metric, symbol Device:R_Small
- added U1: MCP23008-xSS, Package_SO:SSOP-20_5.3x7.2mm_P0.65mm, symbol Interface_Expansion:MCP23008-xSS
Connections:
- wire segments 89 -> 162
- no-connect marks 1 -> 2
Other:
- note added: "I2C Address\n0x20-0x27"
- note added: "RESET"
- note added: "SCL"
- note added: "SDA"
- note removed: "ENC1S"
- note removed: "ENC2S"
- note removed: "PB1"
- note removed: "PB2"
- note removed: "PB3"
- note removed: "PB4"
- moved on the sheet: C1, C2, R1, R2, R3, R4, S2, S3
