File: Breakout_V3/MBRadio_4732_BO3.kicad_pcb (KiCad board)
At the start: 2 copper layers, 65 x 40 mm, 53 parts, among them J3 SJ1-3513-SMT, J4 SJ1-3513-SMT, J5 Conn_01x01_Female, J6 Conn_01x02_Male, J7 Conn_01x09_Male, Q1 Q_NPN_BEC, Q2 Q_NPN_BEC, U1 Si4732-A10, U2 Si4735-D60-GU, U5 TPA301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

Commit message: Add files via upload
Routing:
- net GND: track 45.8 -> 48.7 mm

Commit message: Add files via upload
Parts:
- C10, C11, C15, C9: footprint Capacitor_SMD:C_0402_1005Metric -> Capacitor_SMD:C_0603_1608Metric
- D1: footprint LED_SMD:LED_0402_1005Metric -> LED_SMD:LED_0603_1608Metric_Castellated
- R1, R10, R11, R12, R13, R14, R15, R16, R2, R3, R4, R5, R6, R7, R8, R9: footprint Resistor_SMD:R_0402_1005Metric -> Resistor_SMD:R_0603_1608Metric
- moved R3 2.39 mm to (74.9, 126.9)
- moved R6 2.39 mm to (100.0, 138.0), turned to 0 degrees
- moved R15 2.31 mm to (71.8, 126.9), turned to 0 degrees
- moved R12 2.28 mm to (105.8, 120.0)
- moved R14 1.83 mm to (86.4, 124.5)
- moved R10 1.72 mm to (80.0, 125.7)
- moved R1 1.38 mm to (86.4, 123.0)
- moved R5 1.30 mm to (99.2, 121.2)
- moved C10 1.25 mm to (86.4, 116.8), turned to 180 degrees
- moved C15 1.20 mm to (86.0, 106.1)
- moved R7 1.17 mm to (102.8, 118.7)
- moved C11 1.16 mm to (86.0, 107.7)
- moved R2 1.14 mm to (96.2, 120.8), turned to 180 degrees
- moved R4 0.95 mm to (86.4, 121.5)
- moved R16 0.76 mm to (74.8, 125.4)
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Routing:
- net +3V3: track 73.5 -> 70.5 mm
- net Net-(C12-Pad2): track 4.70 -> 7.63 mm
- net Net-(JP1-Pad1): track 23.6 -> 21.3 mm
- net Net-(R10-Pad1): track 27.6 -> 25.7 mm
- net Net-(R1-Pad2): track 17.4 -> 19.0 mm
- net Net-(C10-Pad1): track 28.4 -> 29.9 mm
- net Net-(J7-Pad3): track 16.4 -> 15.0 mm
- net Net-(R11-Pad1): track 13.1 -> 14.4 mm
- net Net-(C11-Pad1): track 23.3 -> 22.3 mm
- net Net-(R9-Pad1): track 5.98 -> 5.08 mm
- net Net-(C14-Pad2): track 21.3 -> 22.2 mm
- net GND: track 48.7 -> 49.5 mm
- net Net-(C10-Pad2): track 1.47 -> 2.28 mm
- net Net-(J7-Pad5): track 35.4 -> 34.6 mm
- net Net-(C12-Pad1): track 14.6 -> 15.3 mm
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Other:
- board text added: "SI473x BO V3A"
- board text removed: "SI473x BO V3"
