File: Breakout_V3/MBRadio_4732_BO3.sch (KiCad schematic (older format))
At the start: 49 parts, among them J3 SJ1-3513-SMT, J4 SJ1-3513-SMT, J5 Conn_01x01_Female, J6 Conn_01x02_Male, J7 Conn_01x09_Male, Q1 Q_NPN_BEC, Q2 Q_NPN_BEC, U1 Si4732-A10, U2 Si4735-D60-GU, U5 TPA301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

Commit message: Add files via upload
Other:
- note added: "32768Hz TXCO"
- note removed: "32758Hz TXCO"
Changed lines of the file:
@@
 	2050 3050 2050 1650
 Text Notes 650  3000 0    50   Italic 0
-32758Hz TXCO
+32768Hz TXCO
 Wire Wire Line
 	6150 1800 6150 1900

Commit message: Add files via upload
Parts:
- C10, C11, C15, C9: footprint Capacitor_SMD:C_0402_1005Metric -> Capacitor_SMD:C_0603_1608Metric
- D1: footprint LED_SMD:LED_0402_1005Metric -> LED_SMD:LED_0603_1608Metric_Castellated
- R1, R10, R11, R12, R13, R14, R15, R16, R2, R3, R4, R5, R6, R7, R8, R9: footprint Resistor_SMD:R_0402_1005Metric -> Resistor_SMD:R_0603_1608Metric
Changed lines of the file:
@@
 Title "Si4732 BO"
 Date "2021-03-02"
-Rev "Version 3"
+Rev "Version 3A"
 Comp ""
-Comment1 ""
+Comment1 "Convert from 0402->0603 Passives"
 Comment2 "Designed By: Nancy Gail Daniels - AD5EU"
 Comment3 ""
@@
 F 0 "C9" V 9400 4950 50  0000 R CNN
 F 1 "470nF" V 9400 5250 39  0000 R CNN
-F 2 "Capacitor_SMD:C_0402_1005Metric" H 9350 5000 50  0001 C CNN
+F 2 "Capacitor_SMD:C_0603_1608Metric" H 9350 5000 50  0001 C CNN
 F 3 "~" H 9350 5000 50  0001 C CNN
 	1    9350 5000
@@
 F 0 "R3" H 830 3820 50  0000 L CNN
 F 1 "10kΩ" H 960 3600 39  0000 L CNN
-F 2 "Resistor_SMD:R_0402_1005Metric" H 950 3700 50  0001 C CNN
+F 2 "Resistor_SMD:R_0603_1608Metric" H 950 3700 50  0001 C CNN
 F 3 "~" H 950 3700 50  0001 C CNN
 	1    950  3700
@@
 F 0 "R4" H 4590 1400 50  0000 L CNN
 F 1 "4.7kΩ" H 4590 1330 39  0000 L CNN
-F 2 "Resistor_SMD:R_0402_1005Metric" H 4550 1350 50  0001 C CNN
+F 2 "Resistor_SMD:R_0603_1608Metric" H 4550 1350 50  0001 C CNN
 F 3 "~" H 4550 1350 50  0001 C CNN
 	1    4550 1350
@@
 F 0 "R1" H 4290 1400 50  0000 L CNN
 F 1 "4.7kΩ" H 4230 1330 39  0000 L CNN
-F 2 "Resistor_SMD:R_0402_1005Metric" H 4450 1350 50  0001 C CNN
+F 2 "Resistor_SMD:R_0603_1608Metric" H 4450 1350 50  0001 C CNN
 F 3 "~" H 4450 1350 50  0001 C CNN
 	1    4450 1350
@@
 F 0 "D1" H 850 5300 50  0000 L CNN
 F 1 "LED_Small" H 850 5034 50  0001 C CNN
-F 2 "LED_SMD:LED_0402_1005Metric" V 850 5150 50  0001 C CNN
+F 2 "LED_SMD:LED_0603_1608Metric_Castellated" V 850 5150 50  0001 C CNN
 F 3 "~" V 850 5150 50  0001 C CNN
 	1    850  5150
@@
 F 0 "R13" V 2050 7100 50  0000 L CNN
 F 1 "100kΩ" V 2170 7210 39  0000 L CNN
-F 2 "Resistor_SMD:R_0402_1005Metric" H 2100 7300 50  0001 C CNN
+F 2 "Resistor_SMD:R_0603_1608Metric" H 2100 7300 50  0001 C CNN
 F 3 "~" H 2100 7300 50  0001 C CNN
 	1    2100 7300
@@
 F 0 "R5" V 3300 6800 50  0000 L CNN
 F 1 "100kΩ" V 3420 6910 39  0000 L CNN
-F 2 "Resistor_SMD:R_0402_1005Metric" H 3350 7000 50  0001 C CNN
+F 2 "Resistor_SMD:R_0603_1608Metric" H 3350 7000 50  0001 C CNN
 F 3 "~" H 3350 7000 50  0001 C CNN
 	1    3350 7000
@@
 F 0 "R12" V 3300 7000 50  0000 L CNN
 F 1 "100kΩ" V 3420 7110 39  0000 L CNN
-F 2 "Resistor_SMD:R_0402_1005Metric" H 3350 7200 50  0001 C CNN
+F 2 "Resistor_SMD:R_0603_1608Metric" H 3350 7200 50  0001 C CNN
 F 3 "~" H 3350 7200 50  0001 C CNN
 	1    3350 7200
@@
 F 0 "R6" V 950 5450 50  0000 L CNN
 F 1 "1kΩ" V 750 5400 39  0000 L CNN
-F 2 "Resistor_SMD:R_0402_1005Metric" H 850 5450 50  0001 C CNN
+F 2 "Resistor_SMD:R_0603_1608Metric" H 850 5450 50  0001 C CNN
 F 3 "~" H 850 5450 50  0001 C CNN
 	1    850  5450
@@
 F 0 "R7" V 8350 2650 50  0000 L CNN
 F 1 "4.7kΩ" V 8200 2400 39  0000 L CNN
-F 2 "Resistor_SMD:R_0402_1005Metric" H 8300 2550 50  0001 C CNN
+F 2 "Resistor_SMD:R_0603_1608Metric" H 8300 2550 50  0001 C CNN
 F 3 "~" H 8300 2550 50  0001 C CNN
 	1    8300 2550
@@
 F 0 "R8" V 8350 2300 50  0000 L CNN
 F 1 "4.7kΩ" V 8200 2050 39  0000 L CNN
-F 2 "Resistor_SMD:R_0402_1005Metric" H 8300 2200 50  0001 C CNN
+F 2 "Resistor_SMD:R_0603_1608Metric" H 8300 2200 50  0001 C CNN
 F 3 "~" H 8300 2200 50  0001 C CNN
 	1    8300 2200
@@
 F 0 "C10" V 5950 1150 50  0000 R CNN
 F 1 "22nF" V 5850 900 39  0000 R CNN
-F 2 "Capacitor_SMD:C_0402_1005Metric" H 5900 950 50  0001 C CNN
+F 2 "Capacitor_SMD:C_0603_1608Metric" H 5900 950 50  0001 C CNN
 F 3 "~" H 5900 950 50  0001 C CNN
 	1    5900 950
@@
 F 0 "R9" V 2340 2470 50  0000 L CNN
 F 1 "2.0kΩ" V 2230 2290 39  0000 L CNN
-F 2 "Resistor_SMD:R_0402_1005Metric" H 2300 2400 50  0001 C CNN
+F 2 "Resistor_SMD:R_0603_1608Metric" H 2300 2400 50  0001 C CNN
 F 3 "~" H 2300 2400 50  0001 C CNN
 	1    2300 2400
@@
 F 0 "R2" H 1050 2350 50  0000 L CNN
 F 1 "10kΩ" H 1150 2100 39  0000 L CNN
-F 2 "Resistor_SMD:R_0402_1005Metric" H 1150 2200 50  0001 C CNN
+F 2 "Resistor_SMD:R_0603_1608Metric" H 1150 2200 50  0001 C CNN
 F 3 "~" H 1150 2200 50  0001 C CNN
 	1    1150 2200
@@
 F 0 "C11" V 6750 1900 50  0000 R CNN
 F 1 "4.7µF" V 6850 1650 39  0000 R CNN
-F 2 "Capacitor_SMD:C_0402_1005Metric" H 6800 1700 50  0001 C CNN
+F 2 "Capacitor_SMD:C_0603_1608Metric" H 6800 1700 50  0001 C CNN
 F 3 "~" H 6800 1700 50  0001 C CNN
 	1    6800 1700
-	0    -1   1    0
-$EndComp
-$Comp
-L Device:C_Small C15
-U 1 1 607EC8D0
-P 6800 1900
-F 0 "C15" V 6750 2100 50  0000 R CNN
-F 1 "4.7µF" V 6850 1850 39  0000 R CNN
-F 2 "Capacitor_SMD:C_0402_1005Metric" H 6800 1900 50  0001 C CNN
-F 3 "~" H 6800 1900 50  0001 C CNN
-	1    6800 1900
 	0    -1   1    0
 $EndComp
@@
 F 0 "R14" V 5090 3830 50  0000 L CNN
 F 1 "2.0kΩ" V 4980 3640 39  0000 L CNN
-F 2 "Resistor_SMD:R_0402_1005Metric" H 5050 3750 50  0001 C CNN
+F 2 "Resistor_SMD:R_0603_1608Metric" H 5050 3750 50  0001 C CNN
 F 3 "~" H 5050 3750 50  0001 C CNN
 	1    5050 3750
@@
 F 0 "R11" V 5090 3630 50  0000 L CNN
 F 1 "2.0kΩ" V 4980 3440 39  0000 L CNN
-F 2 "Resistor_SMD:R_0402_1005Metric" H 5050 3550 50  0001 C CNN
+F 2 "Resistor_SMD:R_0603_1608Metric" H 5050 3550 50  0001 C CNN
 F 3 "~" H 5050 3550 50  0001 C CNN
 	1    5050 3550
@@
 F 0 "R10" V 5090 4230 50  0000 L CNN
 F 1 "2.0kΩ" V 4980 4040 39  0000 L CNN
-F 2 "Resistor_SMD:R_0402_1005Metric" H 5050 4150 50  0001 C CNN
+F 2 "Resistor_SMD:R_0603_1608Metric" H 5050 4150 50  0001 C CNN
 F 3 "~" H 5050 4150 50  0001 C CNN
 	1    5050 4150
@@
 F 0 "R15" V 2250 2360 50  0000 L CNN
 F 1 "2.0kΩ" V 2370 2530 39  0000 L CNN
-F 2 "Resistor_SMD:R_0402_1005Metric" H 2300 2600 50  0001 C CNN
+F 2 "Resistor_SMD:R_0603_1608Metric" H 2300 2600 50  0001 C CNN
 F 3 "~" H 2300 2600 50  0001 C CNN
 	1    2300 2600
@@
 F 0 "R16" V 5090 4030 50  0000 L CNN
 F 1 "2.0kΩ" V 4980 3840 39  0000 L CNN
-F 2 "Resistor_SMD:R_0402_1005Metric" H 5050 3950 50  0001 C CNN
+F 2 "Resistor_SMD:R_0603_1608Metric" H 5050 3950 50  0001 C CNN
 F 3 "~" H 5050 3950 50  0001 C CNN
 	1    5050 3950
@@
 Wire Wire Line
 	1050 7600 1050 7700
+$Comp
+L Device:C_Small C15
+U 1 1 607EC8D0
+P 6800 1900
+F 0 "C15" V 6750 2100 50  0000 R CNN
+F 1 "4.7µF" V 6850 1850 39  0000 R CNN
+F 2 "Capacitor_SMD:C_0603_1608Metric" H 6800 1900 50  0001 C CNN
+F 3 "~" H 6800 1900 50  0001 C CNN
+	1    6800 1900
+	0    -1   1    0
+$EndComp
 $EndSCHEMATC
